File: STM32H7/BOARD PRJ/renBOOARDv1_STD/renBOOARDv1_STD.kicad_pcb (KiCad board)
At the start: 2 copper layers, 100 x 70 mm, 32 parts, among them U1 STM32H743IITx, U3 TPS54202H, X1 25MHz

Commit message: Avance en USB
Parts:
- removed U2: ~, EasyEDA_Lib:TYPE-C-SMD_TYPE-C-6P
- added C_CK_IN2: 12pF, Capacitor_SMD:C_0402_1005Metric, F.Cu at (175.0, 88.8)
- added F1: Fuse, Fuse:Fuse_1206_3216Metric, F.Cu at (176.9, 89.8)
- added J1: Screw_Terminal_01x02, TerminalBlock:TerminalBlock_MaiXu_MX126-5.0-02P_1x02_P5.00mm, F.Cu at (179.8, 113.5)
- added RCC3: 5.1k, Resistor_SMD:R_0402_1005Metric_Pad0.72x0.64mm_HandSolder, F.Cu at (163.9, 81.2)
- added RCC4: 5.1k, Resistor_SMD:R_0402_1005Metric_Pad0.72x0.64mm_HandSolder, F.Cu at (164.6, 79.5)
- added TVS1: ~, USB_TVS:SOT-23-6_L2.9-W1.6-P0.95-LS2.8-BL, F.Cu at (176.9, 85.0)
- added USB1: ~, USBC_SMD:USB-SMD_USB-TYPE-C-020, F.Cu at (184.0, 85.0)
- moved CREG1_1 19.1 mm to (171.6, 112.3), turned to 0 degrees
- moved RPMUX_2 17.0 mm to (178.0, 101.9), turned to 180 degrees
- moved RPMUX_1 14.7 mm to (177.4, 103.8), turned to -90 degrees
- moved RPMUX_3 13.5 mm to (173.8, 100.3), turned to 0 degrees
- moved PMUX1 13.0 mm to (175.2, 102.1), turned to 0 degrees
- moved C_CK_IN1 11.5 mm to (132.5, 88.0)
- moved C_CK_OUT1 11.5 mm to (126.5, 88.0)
- moved C_VCAP1 11.5 mm to (156.0, 99.5)
- moved C_VCAP2 11.5 mm to (163.5, 77.0)
- moved R_PDR1 11.5 mm to (140.0, 69.4)
- moved U1 11.5 mm to (148.5, 84.5)
- moved X1 11.5 mm to (129.5, 88.0)
- moved RBUCK_1 11.0 mm to (174.8, 105.0)
- moved RBUCK_3 10.6 mm to (172.1, 107.8), turned to -90 degrees
- moved D1 9.67 mm to (173.1, 102.2), turned to 90 degrees
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- renumbered C_CK_OUT2 to C_NRST1
Connections:
- CREG1_2 pad 1: Net-(REG1-VO) -> +3.3V
- REG1 pad 2: Net-(REG1-VO) -> +3.3V
- U1 pad 119: unconnected-(U1-PA8-Pad119) -> /USB_OTG_FS_SOF
- U1 pad 120: unconnected-(U1-PA9-Pad120) -> /USB_OTG_FS_VSBUS
- U1 pad 121: unconnected-(U1-PA10-Pad121) -> /USB_OTG_FS_ID
- U1 pad 122: unconnected-(U1-PA11-Pad122) -> /USB_OTG_FS_D-
- U1 pad 123: unconnected-(U1-PA12-Pad123) -> /USB_OTG_FS_D+
